File: ArduinoShield/ArduinoShield.kicad_pcb (KiCad board)
At the start: 2 copper layers, 47 x 45.7 mm, 45 parts, among them J1 Molex 1053131103, J2 Molex 1053131102, J3 Molex 1053131103, J4 Molex 1053131102, J5 Molex 1053131102, U1 MCP9808_DFN, U2 ALS31300, U3 BME280

Commit message: Small changes to design, added BOM
Parts:
- J_A1: footprint Connector_PinHeader_2.54mm:PinHeader_1x04_P2.54mm_Vertical -> Connector_PinHeader_2.54mm:PinHeader_1x02_P2.54mm_Vertical
- R9: value 470 -> 470R
- moved J_A1 5.08 mm to (112.8, 91.2)
Connections:
- A1 pad 25: A6 -> (no net)
- A1 pad 26: A7 -> (no net)
- J_A1 pad 1: A7 -> A3
- J_A1 pad 2: A6 -> A2
Routing:
- net A6: track 9.33 -> 0.00 mm
- net A7: track 7.02 -> 0.00 mm
Other:
- board text removed: "6"
- board text removed: "7"
