File: ArduinoShield/ArduinoShield.sch (KiCad schematic (older format))
At the start: 41 parts, among them J1 Molex 1053131103, J2 Molex 1053131102, J3 Molex 1053131103, J4 Molex 1053131102, J5 Molex 1053131102, U1 MCP9808_DFN, U2 ALS31300, U3 BME280

Commit message: Small changes to design, added BOM
Parts:
- removed J_A1: J_A, Connector_PinHeader_2.54mm:PinHeader_1x04_P2.54mm_Vertical, symbol Connector_Generic:Conn_01x04
- added J_A1: J_A, Connector_PinHeader_2.54mm:PinHeader_1x02_P2.54mm_Vertical, symbol Connector_Generic:Conn_01x02
- R9: value 470 -> 470R
Connections:
- net A2: now also J_A1.2 (Pin_2)
- net A3: now also J_A1.1 (Pin_1)
- net A6: no longer names the net of A1.25 (A6)
- net A7: no longer names the net of A1.26 (A7)
Changed lines of the file:
@@
 	2350 5300 2100 5300
 Connection ~ 2350 5850
-Connection ~ 2350 5300
 Text GLabel 8850 2500 0    50   Input ~ 0
 DFlow
 Wire Wire Line
 	9050 2500 8850 2500
-Text GLabel 2100 4950 1    50   Input ~ 0
-DFlow
 $Comp
 L Diode:MM3Zxx D1
@@
 	1    0    0    -1
 $EndComp
-$Comp
-L Device:R R9
-U 1 1 5E71C48D
-P 2500 5300
-F 0 "R9" H 2570 5346 50  0000 L CNN
-F 1 "470" H 2570 5255 50  0000 L CNN
-F 2 "Resistor_SMD:R_0201_0603Metric" V 2430 5300 50  0001 C CNN
-F 3 "~" H 2500 5300 50  0001 C CNN
-	1    2500 5300
-	0    -1   -1   0
-$EndComp
-Wire Wire Line
-	2650 5300 2750 5300
-Wire Wire Line
-	2100 4950 2100 5300
-Connection ~ 2100 5300
 Wire Wire Line
 	3550 3700 3600 3700
@@
 Wire Wire Line
 	10050 2400 10400 2400
-Wire Wire Line
-	10050 2700 10400 2700
-Wire Wire Line
-	10050 2800 10400 2800
 Text GLabel 10400 2300 2    50   Input ~ 0
 A2
 Text GLabel 10400 2400 2    50   Input ~ 0
 A3
-Text GLabel 10400 2700 2    50   Input ~ 0
-A6
-Text GLabel 10400 2800 2    50   Input ~ 0
-A7
 Wire Notes Line
 	7400 500  8300 500
 Wire Notes Line
 	7400 2500 7400 500
-$Comp
-L Connector_Generic:Conn_01x04 J_A1
-U 1 1 5E87F739
-P 8050 800
-F 0 "J_A1" H 8000 1000 50  0000 L CNN
-F 1 "J_A" V 8200 500 50  0000 L CNN
-F 2 "Connector_PinHeader_2.54mm:PinHeader_1x04_P2.54mm_Vertical" H 8050 800 50  0001 C CNN
-F 3 "~" H 8050 800 50  0001 C CNN
-	1    8050 800
-	1    0    0    -1
-$EndComp
-Text GLabel 7750 800  0    50   Input ~ 0
-A6
-Text GLabel 7750 700  0    50   Input ~ 0
-A7
-Text GLabel 7750 1000 0    50   Input ~ 0
+Text GLabel 7800 900  0    50   Input ~ 0
 A2
-Text GLabel 7750 900  0    50   Input ~ 0
+Text GLabel 7800 800  0    50   Input ~ 0
 A3
 Wire Wire Line
-	7750 700  7850 700
-Wire Wire Line
-	7750 800  7850 800
-Wire Wire Line
-	7850 900  7750 900
-Wire Wire Line
-	7750 1000 7850 1000
+	7900 800  7800 800
+Wire Wire Line
+	7800 900  7900 900
 Text Notes 7450 2450 0    50   ~ 0
 Headers
@@
 	7900 2150 7900 2200
 Connection ~ 7900 2150
+Text GLabel 2100 4950 1    50   Input ~ 0
+DFlow
+Connection ~ 2100 5300
+Wire Wire Line
+	2100 4950 2100 5300
+Wire Wire Line
+	2650 5300 2750 5300
+Connection ~ 2350 5300
+$Comp
+L Device:R R9
+U 1 1 5E71C48D
+P 2500 5300
+F 0 "R9" H 2570 5346 50  0000 L CNN
+F 1 "470R" H 2570 5255 50  0000 L CNN
+F 2 "Resistor_SMD:R_0201_0603Metric" V 2430 5300 50  0001 C CNN
+F 3 "~" H 2500 5300 50  0001 C CNN
+	1    2500 5300
+	0    -1   -1   0
+$EndComp
+$Comp
+L Connector_Generic:Conn_01x02 J_A1
+U 1 1 5E898E60
+P 8100 800
+F 0 "J_A1" H 8018 593 50  0000 C CNN
+F 1 "J_A" V 8200 800 50  0000 C CNN
+F 2 "Connector_PinHeader_2.54mm:PinHeader_1x02_P2.54mm_Vertical" H 8100 800 50  0001 C CNN
+F 3 "~" H 8100 800 50  0001 C CNN
+	1    8100 800
+	1    0    0    -1
+$EndComp
 $EndSCHEMATC

Commit message: Updated Hole size for Arduino, Created Footprint for bigger hole sizes
Parts:
- A1: footprint Module:Arduino_Nano -> ArduinoShield:Arduino_Nano
Changed lines of the file:
@@
 F 0 "A1" H 9550 1011 50  0000 C CNN
 F 1 "Arduino_Nano_v3.x" H 9550 920 50  0000 C CNN
-F 2 "Module:Arduino_Nano" H 9550 2100 50  0001 C CIN
+F 2 "ArduinoShield:Arduino_Nano" H 9550 2100 50  0001 C CIN
 F 3 "http://www.mouser.com/pdfdocs/Gravitech_Arduino_Nano3_0.pdf" H 9550 2100 50  0001 C CNN
 	1    9550 2100

Commit message: Modified part that was wrong in KiCad Library (MCP9808)
Parts:
- U1: footprint Package_DFN_QFN:DFN-8-1EP_3x3mm_P0.65mm_EP1.55x2.4mm -> Package_DFN_QFN:DFN-8-1EP_3x2mm_P0.5mm_EP1.3x1.5mm
Changed lines of the file:
@@
 Comment4 ""
 $EndDescr
-$Comp
-L ArduinoEnivronmentShield:MCP9808_DFN U1
-U 1 1 5E6BD66B
-P 1800 1650
-F 0 "U1" H 2244 1696 50  0000 L CNN
-F 1 "MCP9808_DFN" H 1969 1181 50  0000 L CNN
-F 2 "Package_DFN_QFN:DFN-8-1EP_3x3mm_P0.65mm_EP1.55x2.4mm" H 700 1150 50  0001 C CNN
-F 3 "http://ww1.microchip.com/downloads/en/DeviceDoc/22203b.pdf" H 1550 2100 50  0001 C CNN
-	1    1800 1650
-	1    0    0    -1
-$EndComp
 Wire Wire Line
 	1800 2150 1850 2150
@@
 	1    0    0    -1
 $EndComp
+$Comp
+L ArduinoEnivronmentShield:MCP9808_DFN U1
+U 1 1 5E6BD66B
+P 1800 1650
+F 0 "U1" H 2244 1696 50  0000 L CNN
+F 1 "MCP9808_DFN" H 1969 1181 50  0000 L CNN
+F 2 "Package_DFN_QFN:DFN-8-1EP_3x2mm_P0.5mm_EP1.3x1.5mm" H 700 1150 50  0001 C CNN
+F 3 "http://ww1.microchip.com/downloads/en/DeviceDoc/22203b.pdf" H 1550 2100 50  0001 C CNN
+	1    1800 1650
+	1    0    0    -1
+$EndComp
